Commit message: add ${prefix} to material name in urdf for multi-robot

File: iiwa_description/urdf/iiwa.urdf.xacro (robot description, xacro)
@@ -2,5 +2,5 @@
 <robot xmlns:xacro="http://www.ros.org/wiki/xacro">
   <xacro:macro name="iiwa" params="parent prefix *origin">
-  <material name="gray">
+  <material name="${prefix}gray">
     <color rgba="0.5 0.5 0.5 1.0"/>
   </material>
@@ -152,5 +152,5 @@
       <visual>
         <origin rpy="0 0 0" xyz="0 0 0.07"/>
-        <material name="gray"/>
+        <material name="${prefix}gray"/>
         <geometry>
           <mesh filename="package://iiwa_description/meshes/lbr_iiwa_14_r820/visual/link_7_2.stl" scale ="0.001 0.001 0.001"/>
